Commit message: Standardize YuLong component and joint names

File: Assets/remake5/urdf/remake5.urdf (robot description, URDF)
Before this commit: robot remake5, 13 links, 12 joints
Links:
- removed link controller
- removed link dabi
- removed link huosai2a
- removed link huosai2b
- removed link huosai3a
- removed link huosai3b
- removed link huosai4a
- removed link huosai4b
- removed link sigan1
- removed link sigan2
- removed link watou
- removed link xiaobi
- added link boom, mass 11.1002972149815; collision mesh filename=package://remake5/meshes/dabi.STL; visual mesh filename=package://remake5/meshes/dabi.STL
- added link boom_cylinder_barrel, mass 0.656016306211451; collision mesh filename=package://remake5/meshes/huosai2a.STL; visual mesh filename=package://remake5/meshes/huosai2a.STL
- added link boom_cylinder_rod, mass 1.53242458264255; collision mesh filename=package://remake5/meshes/huosai2b.STL; visual mesh filename=package://remake5/meshes/huosai2b.STL
- added link bucket, mass 6.72063953784663; collision mesh filename=package://remake5/meshes/watou.STL; visual mesh filename=package://remake5/meshes/watou.STL
- added link bucket_bellcrank, mass 0.873348986641261; collision mesh filename=package://remake5/meshes/sigan2.STL; visual mesh filename=package://remake5/meshes/sigan2.STL
- added link bucket_cylinder_barrel, mass 1.11193350717462; collision mesh filename=package://remake5/meshes/huosai4a.STL; visual mesh filename=package://remake5/meshes/huosai4a.STL
- added link bucket_cylinder_rod, mass 0.584099353233864; collision mesh filename=package://remake5/meshes/huosai4b.STL; visual mesh filename=package://remake5/meshes/huosai4b.STL
- added link bucket_link, mass 0.766349887273834; collision mesh filename=package://remake5/meshes/sigan1.STL; visual mesh filename=package://remake5/meshes/sigan1.STL
- added link stick, mass 4.97678856772179; collision mesh filename=package://remake5/meshes/xiaobi.STL; visual mesh filename=package://remake5/meshes/xiaobi.STL
- added link stick_cylinder_barrel, mass 1.2043; collision mesh filename=package://remake5/meshes/huosai3a.STL; visual mesh filename=package://remake5/meshes/huosai3a.STL
- added link stick_cylinder_rod, mass 0.636593414100438; collision mesh filename=package://remake5/meshes/huosai3b.STL; visual mesh filename=package://remake5/meshes/huosai3b.STL
- added link upper_structure, mass 77.6129571793414; collision mesh filename=package://remake5/meshes/controller.STL; visual mesh filename=package://remake5/meshes/controller.STL
Joints:
- removed joint base_to_controller_joint
- removed joint controller_to_dabi_joint
- removed joint controller_to_huosai2a_joint
- removed joint dabi_to_huosai2b_joint
- removed joint dabi_to_huosai3a_joint
- removed joint dabi_to_xiaobi_joint
- removed joint sigan2_to_huosai4b_joint
- removed joint watou_to_sigan1
- removed joint xiaobi_to_huosai3b_joint
- removed joint xiaobi_to_huosai4a
- removed joint xiaobi_to_sigan2_joint
- removed joint xiaobi_to_watou_joint
- added joint boom_joint: type revolute, parent upper_structure, child boom, origin xyz=0.84031 -0.1344 -0.224 rpy=0 0 0, axis 0 1 0, limit lower=-3.14 upper=3.14 effort=100 velocity=1
- added joint boom_to_boom_cylinder_rod_joint: type revolute, parent boom, child boom_cylinder_rod, origin xyz=0.174394120072099 0.0569999650974322 0.998450892564747 rpy=0 0 0, axis 0 -0.99999999999998 0, limit lower=-3.14 upper=3.14 effort=100 velocity=1
- added joint boom_to_stick_cylinder_barrel_joint: type revolute, parent boom, child stick_cylinder_barrel, origin xyz=0.330116693603899 0.0574999339313985 1.36767977838426 rpy=0 0 0, axis 0 -0.99999999999998 0, limit lower=-3.14 upper=3.14 effort=100 velocity=1
- added joint bucket_bellcrank_to_bucket_cylinder_rod_joint: type revolute, parent bucket_bellcrank, child bucket_cylinder_rod, origin xyz=0.142616525247579 -0.0590000285429868 0.109820414121545 rpy=0 0 0, axis 0 0.99999999999998 0, limit lower=-3.14 upper=3.14 effort=100 velocity=1
- added joint bucket_joint: type revolute, parent stick, child bucket, origin xyz=0.455946627104724 -0.00650009125267029 -0.827736395860433 rpy=0 0 0, axis 0 0.99999999999998 0, limit lower=-3.14 upper=3.14 effort=100 velocity=1
- added joint bucket_to_bucket_link_joint: type revolute, parent bucket, child bucket_link, origin xyz=0.0997753251526592 0 0.00667390709543314 rpy=0 0 0, axis 0 0.99999999999998 0, limit lower=-3.14 upper=3.14 effort=100 velocity=1
- added joint stick_joint: type revolute, parent boom, child stick, origin xyz=1.09359335696479 0.123999781129014 1.47352591557926 rpy=0 0 0, axis 0 0.99999999999998 0, limit lower=-3.14 upper=3.14 effort=100 velocity=1
- added joint stick_to_bucket_bellcrank_joint: type revolute, parent stick, child bucket_bellcrank, origin xyz=0.416378305836035 -0.0100000833334549 -0.755908524273468 rpy=0 0 0, axis 0 -0.99999999999998 0, limit lower=-3.14 upper=3.14 effort=100 velocity=1
- added joint stick_to_bucket_cylinder_barrel_joint: type revolute, parent stick, child bucket_cylinder_barrel, origin xyz=0.262116942692277 -0.0665000514603171 -0.092419584883574 rpy=0 0 0, axis 0 -0.99999999999998 0, limit lower=-3.14 upper=3.14 effort=100 velocity=1
- added joint stick_to_stick_cylinder_rod_joint: type revolute, parent stick, child stick_cylinder_rod, origin xyz=-0.0011748 -0.069 0.198 rpy=0 0 0, axis 0 -1 0, limit lower=-3.14 upper=3.14 effort=100 velocity=1
- added joint swing_joint: type revolute, parent base_link, child upper_structure, origin xyz=0 0 0.67 rpy=0 0 0, axis 0 0 -1, limit lower=-3.14 upper=3.14 effort=100 velocity=1
- added joint upper_structure_to_boom_cylinder_barrel_joint: type revolute, parent upper_structure, child boom_cylinder_barrel, origin xyz=0.695305211935226 -0.0768994271774273 0.00399999238143445 rpy=0 0 0, axis 0 -0.99999999999998 0, limit lower=-3.14 upper=3.14 effort=100 velocity=1
